Commit message: 为机器日修改了一些参数，添加了五个激光雷达

File: src/whc_description/urdf/whc_description.urdf (robot description, URDF)
Before this commit: robot whc, 8 links, 7 joints
Links:
- added link base_footprint
- added link left_wheel_back, mass 500.0; collision cylinder length=0.3 radius=0.48; visual cylinder length=0.3 radius=0.48
- added link left_wheel_front, mass 500.0; collision cylinder length=0.3 radius=0.48; visual cylinder length=0.3 radius=0.48
- added link left_wheel_middle, mass 500.0; collision cylinder length=0.3 radius=0.48; visual cylinder length=0.3 radius=0.48
- added link left_wheel_middle1, mass 500.0; collision cylinder length=0.3 radius=0.48; visual cylinder length=0.3 radius=0.48
- added link left_wheel_middle2, mass 500.0; collision cylinder length=0.3 radius=0.48; visual cylinder length=0.3 radius=0.48
- added link right_wheel_back, mass 500.0; collision cylinder length=0.3 radius=0.48; visual cylinder length=0.3 radius=0.48
- added link right_wheel_front, mass 500.0; collision cylinder length=0.3 radius=0.48; visual cylinder length=0.3 radius=0.48
- added link right_wheel_middle, mass 500.0; collision cylinder length=0.3 radius=0.48; visual cylinder length=0.3 radius=0.48
- added link right_wheel_middle1, mass 500.0; collision cylinder length=0.3 radius=0.48; visual cylinder length=0.3 radius=0.48
- added link right_wheel_middle2, mass 500.0; collision cylinder length=0.3 radius=0.48; visual cylinder length=0.3 radius=0.48
Joints:
- added joint base_footprint_joint: type fixed, parent base_footprint, child base_link, origin xyz=0 0 0 rpy=0 0 0
- added joint left_wheel_back_joint: type continuous, parent base_link, child left_wheel_back, origin xyz=-2.0 1.4 0.47 rpy=0 0 0, axis 0 1 0
- added joint left_wheel_front_joint: type continuous, parent base_link, child left_wheel_front, origin xyz=2.0 1.4 0.47 rpy=0 0 0, axis 0 1 0
- added joint left_wheel_middle1_joint: type continuous, parent base_link, child left_wheel_middle1, origin xyz=1 1.4 0.47 rpy=0 0 0, axis 0 1 0
- added joint left_wheel_middle2_joint: type continuous, parent base_link, child left_wheel_middle2, origin xyz=-1 1.4 0.47 rpy=0 0 0, axis 0 1 0
- added joint left_wheel_middle_joint: type continuous, parent base_link, child left_wheel_middle, origin xyz=0 1.4 0.47 rpy=0 0 0, axis 0 1 0
- added joint right_wheel_back_joint: type continuous, parent base_link, child right_wheel_back, origin xyz=-2.0 -1.4 0.47 rpy=0 0 0, axis 0 1 0
- added joint right_wheel_front_joint: type continuous, parent base_link, child right_wheel_front, origin xyz=2.0 -1.4 0.47 rpy=0 0 0, axis 0 1 0
- added joint right_wheel_middle1_joint: type continuous, parent base_link, child right_wheel_middle1, origin xyz=1 -1.4 0.47 rpy=0 0 0, axis 0 1 0
- added joint right_wheel_middle2_joint: type continuous, parent base_link, child right_wheel_middle2, origin xyz=-1 -1.4 0.47 rpy=0 0 0, axis 0 1 0
- added joint right_wheel_middle_joint: type continuous, parent base_link, child right_wheel_middle, origin xyz=0 -1.4 0.47 rpy=0 0 0, axis 0 1 0

File: src/whc_description/urdf/whc_description_gazebo.xacro (robot description, xacro)
@@ -1,4 +1,10 @@
 <?xml version="1.0" encoding="utf-8"?>
 <robot name="whc" xmlns:xacro="http://ros.org/wiki/xacro">
+  <link name="base_footprint"/>
+  <joint name="base_footprint_joint" type="fixed">
+    <parent link="base_footprint"/>
+    <child link="base_link"/>
+    <origin xyz="0 0 0" rpy="0 0 0"/>
+  </joint>
   <link name="base_link">
     <inertial>
@@ -15,5 +21,5 @@
       </geometry>
       <material name="">
-        <color rgba="0.792 0.820 0.933 1"/>
+        <color rgba="0.5 0.5 0.5 1"/>
       </material>
     </visual>
@@ -25,35 +31,4 @@
     </collision>
   </link>
-  <!-- 激光雷达链接 - 安装在机器人底部 -->
-  <!--link name="lidar_link">
-    <inertial>
-      <mass value="0.5"/>
-      <origin xyz="0 0 0"/>
-      <inertia ixx="0.001" ixy="0.0" ixz="0.0"
-               iyy="0.001" iyz="0.0"
-               izz="0.001"/>
-    </inertial>
-    <visual>
-      <origin xyz="0 0 0" rpy="0 0 0"/>
-      <geometry>
-        <cylinder radius="0.1" length="0.05"/>
-      </geometry>
-      <material name="">
-        <color rgba="0.2 0.2 0.8 0.8"/>
-      </material>
-    </visual>
-    <collision>
-      <origin xyz="0 0 0" rpy="0 0 0"/>
-      <geometry>
-        <cylinder radius="0.1" length="0.05"/>
-      </geometry>
-    </collision>
-  </link-->
-<!-- 激光雷达关节 - 固定连接到base_link底部 -->
-<!--joint name="lidar_joint" type="fixed">
-  <parent link="base_link"/>
-  <child link="lidar_link"/>
-  <origin xyz="0 0 1.3" rpy="0 0 0"/>
-</joint-->
   <link name="left_wheel_back">
     <inertial>
@@ -70,15 +45,15 @@
       </geometry>
       <material name="">
-        <color rgba="0.792 0.820 0.933 1"/>
-      </material>
-    </visual>
-    <collision>
-      <origin xyz="0 0 0" rpy="1.5708 0 0"/>
-      <geometry>
-        <cylinder length="0.3" radius="0.48"/>
-      </geometry>
-    </collision>
-  </link>
-    <link name="left_wheel_middle">
+        <color rgba="0.5 0.5 0.5 1"/>
+      </material>
+    </visual>
+    <collision>
+      <origin xyz="0 0 0" rpy="1.5708 0 0"/>
+      <geometry>
+        <cylinder length="0.3" radius="0.48"/>
+      </geometry>
+    </collision>
+  </link>
+  <link name="left_wheel_middle">
     <inertial>
       <mass value="500.0"/>
@@ -94,5 +69,5 @@
       </geometry>
       <material name="">
-        <color rgba="0.792 0.820 0.933 1"/>
+        <color rgba="0.5 0.5 0.5 1"/>
       </material>
     </visual>
@@ -118,5 +93,5 @@
       </geometry>
       <material name="">
-        <color rgba="0.792 0.820 0.933 1"/>
+        <color rgba="0.5 0.5 0.5 1"/>
       </material>
     </visual>
@@ -142,5 +117,5 @@
       </geometry>
       <material name="">
-        <color rgba="0.792 0.820 0.933 1"/>
+        <color rgba="0.5 0.5 0.5 1"/>
       </material>
     </visual>
@@ -385,5 +360,5 @@
       </geometry>
       <material name="">
-        <color rgba="0.792 0.820 0.933 1"/>
+        <color rgba="0.5 0.5 0.5 1"/>
       </material>
     </visual>
@@ -416,5 +391,5 @@
       </geometry>
       <material name="">
-        <color rgba="0.792 0.820 0.933 1"/>
+        <color rgba="0.5 0.5 0.5 1"/>
       </material>
     </visual>
@@ -447,5 +422,5 @@
       </geometry>
       <material name="">
-        <color rgba="1 0 0 1"/>
+        <color rgba="0.5 0.5 0.5 1"/>
       </material>
     </visual>
@@ -478,5 +453,5 @@
       </geometry>
       <material name="">
-        <color rgba="0.792 0.820 0.933 1"/>
+        <color rgba="0.5 0.5 0.5 1"/>
       </material>
     </visual>
@@ -509,5 +484,5 @@
       </geometry>
       <material name="">
-        <color rgba="0.792 0.820 0.933 1"/>
+        <color rgba="0.5 0.5 0.5 1"/>
       </material>
     </visual>
@@ -540,5 +515,5 @@
       </geometry>
       <material name="">
-        <color rgba="0.792 0.820 0.933 1"/>
+        <color rgba="0.5 0.5 0.5 1"/>
       </material>
     </visual>
@@ -571,5 +546,5 @@
       </geometry>
       <material name="">
-        <color rgba="0.1 0.1 0.1 1"/>
+        <color rgba="0.5 0.5 0.5 1"/>
       </material>
     </visual>
@@ -604,5 +579,5 @@
       </geometry>
       <material name="global_cam_material">
-        <color rgba="0.8 0.2 0.2 0.8"/>
+        <color rgba="0.5 0.5 0.5 1"/>
       </material>
     </visual>
@@ -1159,3 +1134,83 @@
     </sensor>
   </gazebo>
+  <!-- 包含激光雷达宏及实例化 -->
+  <xacro:property name="PI" value="3.14159265359"/>
+  <!-- ==================== 3D LiDAR Sensors ==================== -->
+  <xacro:macro name="lidar_3d_fov" params="prefix x y z yaw">
+    <link name="${prefix}_link">
+      <visual>
+        <geometry>
+          <cylinder radius="0.03" length="0.05"/>
+        </geometry>
+        <material name="${prefix}_color">
+          <color rgba="0.9 0.1 0.1 1.0"/>
+        </material>
+      </visual>
+      <collision>
+        <geometry>
+          <cylinder radius="0.03" length="0.05"/>
+        </geometry>
+      </collision>
+      <inertial>
+        <mass value="0.05"/>
+        <inertia ixx="0.00001" ixy="0" ixz="0" iyy="0.00001" iyz="0" izz="0.00001"/>
+      </inertial>
+    </link>
+    <joint name="${prefix}_joint" type="fixed">
+      <parent link="base_link"/>
+      <child link="${prefix}_link"/>
+      <origin xyz="${x} ${y} ${z}" rpy="0 0 ${yaw}"/>
+    </joint>
+    <gazebo reference="${prefix}_link">
+      <material>Gazebo/Red</material>
+      <sensor type="ray" name="${prefix}_sensor">
+        <pose>0 0 0 0 0 0</pose>
+        <visualize>false</visualize>
+        <update_rate>10</update_rate>
+        <ray>
+          <scan>
+            <horizontal>
+              <samples>180</samples>
+              <resolution>1</resolution>
+              <min_angle>${-PI/2}</min_angle>
+              <max_angle>${PI/2}</max_angle>
+            </horizontal>
+            <vertical>
+              <samples>8</samples>
+              <resolution>1</resolution>
+              <min_angle>${-15.0*PI/180.0}</min_angle>
+              <max_angle>${15.0*PI/180.0}</max_angle>
+            </vertical>
+          </scan>
+          <range>
+            <min>0.1</min>
+            <max>30.0</max>
+            <resolution>0.01</resolution>
+          </range>
+          <noise>
+            <type>gaussian</type>
+            <mean>0.0</mean>
+            <stddev>0.005</stddev>
+          </noise>
+        </ray>
+        <plugin name="${prefix}_plugin" filename="libgazebo_ros_ray_sensor.so">
+          <ros>
+            <remapping>~/out:=${prefix}/points</remapping>
+          </ros>
+          <output_type>sensor_msgs/PointCloud2</output_type>
+          <frame_name>${prefix}_link</frame_name>
+        </plugin>
+      </sensor>
+    </gazebo>
+  </xacro:macro>
+  <!-- lidar_1: 后 -->
+  <xacro:lidar_3d_fov prefix="lidar_1" x="-2.5" y="0" z="1.5" yaw="${PI}"/>
+  <!-- lidar_2: 左 -->
+  <xacro:lidar_3d_fov prefix="lidar_2" x="0" y="1.8" z="1.5" yaw="${PI/2}"/>
+  <!-- lidar_3: 前左 -->
+  <xacro:lidar_3d_fov prefix="lidar_3" x="2.5" y="1.4" z="1.5" yaw="${PI/4}"/>
+  <!-- lidar_4: 前右 -->
+  <xacro:lidar_3d_fov prefix="lidar_4" x="2.5" y="-1.4" z="1.5" yaw="${-PI/4}"/>
+  <!-- lidar_5: 右 -->
+  <xacro:lidar_3d_fov prefix="lidar_5" x="0" y="-1.8" z="1.5" yaw="${-PI/2}"/>
 </robot>
